File: groundwork/Vim/new_pcb/arm_pcb/arm_pcb.kicad_sch (KiCad schematic)
At the start: 18 parts, among them U1 NODEMCU32S

Commit message: pcb schematic udpate final v0.1
Connections:
- net SPI_MISO: now also MotorDriver4.3 (Pin_3)
- net SPI_MOSI: now also MotorDriver4.2 (Pin_2)
- net SPI_SCK: now also MotorDriver4.4 (Pin_4), Stepper1.1 (Pin_1); no longer MotorDriver4.5 (Pin_5)
- net at U1.GPIO5: now also MotorDriver3.5 (Pin_5); no longer Stepper1.1 (Pin_1)
- net at U1.GPIO27: now also MotorDriver3.3 (Pin_3); no longer EncoderA1.2 (Pin_2)
- net at U1.GPIO9: no longer MotorDriver3.3 (Pin_3)
- net at MotorDriver3.4 (Pin_4): now also U1.GPIO15; no longer U1.GPIO10
- net at U1.GPIO11: no longer MotorDriver3.5 (Pin_5)
- net a_in_3: now reaches EncoderA3.2 (Pin_2)
- net a_in_3: now also U1.GPIO36; no longer U1.GPIO0
- net a_in_4: now reaches EncoderA4.2 (Pin_2)
- net a_in_4: now also U1.GPIO39; no longer U1.GPIO15
- net m4_4: now reaches U1.GPIO2
- net m4_4: now also MotorDriver4.5 (Pin_5)
- net servo3: now reaches I2Cbreakout1.3 (Pin_3), U1.GPIO21
- net servo3: now also Servo3.2 (Pin_2)
- net servo4: now reaches I2Cbreakout1.4 (Pin_4), U1.GPIO22
- net servo4: now also Servo4.2 (Pin_2)
- net a_in_1: now reaches U1.GPIO34
- net a_in_1: now also EncoderA1.2 (Pin_2); no longer MotorDriver1.2 (Pin_2)
- net a_in_2: now reaches U1.GPIO35
- net a_in_2: now also EncoderA2.2 (Pin_2); no longer MotorDriver1.3 (Pin_3)
- net m1_2: now reaches U1.GPIO4
- net m1_2: now also MotorDriver1.3 (Pin_3); no longer EncoderA2.2 (Pin_2)
- net at U1.GPIO6: no longer MotorDriver4.4 (Pin_4)
- net at U1.GPIO7: no longer Servo4.2 (Pin_2)
- net at U1.GPIO8: no longer Servo3.2 (Pin_2)
- new net m1_1: MotorDriver1.2 (Pin_2), U1.GPIO0

Commit message: final pcb v0.2
Parts:
- EncoderA1, EncoderA2, EncoderA3, EncoderA4, Servo1, Servo2, Servo3, Servo4, Stepper1, Stepper_GND1: footprint Connector_JST:JST_XA_B03B-XASK-1-A_1x03_P2.50mm_Vertical -> Connector_JST:JST_XH_B3B-XH-A_1x03_P2.50mm_Vertical
- I2Cbreakout1, UART0breakout1: footprint Connector_JST:JST_XA_B04B-XASK-1-A_1x04_P2.50mm_Vertical -> Connector_JST:JST_XH_B4B-XH-A_1x04_P2.50mm_Vertical
- MotorDriver1, MotorDriver2, MotorDriver3, MotorDriver4: footprint Connector_JST:JST_XA_B05B-XASK-1-A_1x05_P2.50mm_Vertical -> Connector_JST:JST_XH_B5B-XH-A_1x05_P2.50mm_Vertical
Changed lines of the file:
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@@
       (effects (font (size 1.27 1.27)) (justify right))
     )
-    (property "Footprint" "Connector_JST:JST_XA_B03B-XASK-1-A_1x03_P2.50mm_Vertical" (at 182.88 93.98 0)
+    (property "Footprint" "Connector_JST:JST_XH_B3B-XH-A_1x03_P2.50mm_Vertical" (at 182.88 93.98 0)
       (effects (font (size 1.27 1.27)) hide)
     )
@@
       (effects (font (size 1.27 1.27)))
     )
-    (property "Footprint" "Connector_JST:JST_XA_B05B-XASK-1-A_1x05_P2.50mm_Vertical" (at 43.18 85.09 0)
+    (property "Footprint" "Connector_JST:JST_XH_B5B-XH-A_1x05_P2.50mm_Vertical" (at 43.18 85.09 0)
       (effects (font (size 1.27 1.27)) hide)
     )
@@
       (effects (font (size 1.27 1.27)) (justify right))
     )
-    (property "Footprint" "Connector_JST:JST_XA_B03B-XASK-1-A_1x03_P2.50mm_Vertical" (at 170.18 81.28 0)
+    (property "Footprint" "Connector_JST:JST_XH_B3B-XH-A_1x03_P2.50mm_Vertical" (at 170.18 81.28 0)
       (effects (font (size 1.27 1.27)) hide)
     )
@@
       (effects (font (size 1.27 1.27)) (justify right))
     )
-    (property "Footprint" "Connector_JST:JST_XA_B04B-XASK-1-A_1x04_P2.50mm_Vertical" (at 207.01 90.17 0)
+    (property "Footprint" "Connector_JST:JST_XH_B4B-XH-A_1x04_P2.50mm_Vertical" (at 207.01 90.17 0)
       (effects (font (size 1.27 1.27)) hide)
     )
@@
       (effects (font (size 1.27 1.27)) (justify right))
     )
-    (property "Footprint" "Connector_JST:JST_XA_B03B-XASK-1-A_1x03_P2.50mm_Vertical" (at 167.64 68.58 0)
+    (property "Footprint" "Connector_JST:JST_XH_B3B-XH-A_1x03_P2.50mm_Vertical" (at 167.64 68.58 0)
       (effects (font (size 1.27 1.27)) hide)
     )
@@
       (effects (font (size 1.27 1.27)))
     )
-    (property "Footprint" "Connector_JST:JST_XA_B03B-XASK-1-A_1x03_P2.50mm_Vertical" (at 252.73 66.04 0)
+    (property "Footprint" "Connector_JST:JST_XH_B3B-XH-A_1x03_P2.50mm_Vertical" (at 252.73 66.04 0)
       (effects (font (size 1.27 1.27)) hide)
     )
@@
       (effects (font (size 1.27 1.27)))
     )
-    (property "Footprint" "Connector_JST:JST_XA_B03B-XASK-1-A_1x03_P2.50mm_Vertical" (at 100.33 134.62 0)
+    (property "Footprint" "Connector_JST:JST_XH_B3B-XH-A_1x03_P2.50mm_Vertical" (at 100.33 134.62 0)
       (effects (font (size 1.27 1.27)) hide)
     )
@@
       (effects (font (size 1.27 1.27)))
     )
-    (property "Footprint" "Connector_JST:JST_XA_B05B-XASK-1-A_1x05_P2.50mm_Vertical" (at 43.18 105.41 0)
+    (property "Footprint" "Connector_JST:JST_XH_B5B-XH-A_1x05_P2.50mm_Vertical" (at 43.18 105.41 0)
       (effects (font (size 1.27 1.27)) hide)
     )
@@
       (effects (font (size 1.27 1.27)))
     )
-    (property "Footprint" "Connector_JST:JST_XA_B03B-XASK-1-A_1x03_P2.50mm_Vertical" (at 137.16 134.62 0)
+    (property "Footprint" "Connector_JST:JST_XH_B3B-XH-A_1x03_P2.50mm_Vertical" (at 137.16 134.62 0)
       (effects (font (size 1.27 1.27)) hide)
     )
@@
       (effects (font (size 1.27 1.27)))
     )
-    (property "Footprint" "Connector_JST:JST_XA_B03B-XASK-1-A_1x03_P2.50mm_Vertical" (at 119.38 134.62 0)
+    (property "Footprint" "Connector_JST:JST_XH_B3B-XH-A_1x03_P2.50mm_Vertical" (at 119.38 134.62 0)
       (effects (font (size 1.27 1.27)) hide)
     )
@@
       (effects (font (size 1.27 1.27)) (justify right))
     )
-    (property "Footprint" "Connector_JST:JST_XA_B03B-XASK-1-A_1x03_P2.50mm_Vertical" (at 184.15 125.73 0)
+    (property "Footprint" "Connector_JST:JST_XH_B3B-XH-A_1x03_P2.50mm_Vertical" (at 184.15 125.73 0)
       (effects (font (size 1.27 1.27)) hide)
     )
@@
       (effects (font (size 1.27 1.27)))
     )
-    (property "Footprint" "Connector_JST:JST_XA_B05B-XASK-1-A_1x05_P2.50mm_Vertical" (at 43.18 63.5 0)
+    (property "Footprint" "Connector_JST:JST_XH_B5B-XH-A_1x05_P2.50mm_Vertical" (at 43.18 63.5 0)
       (effects (font (size 1.27 1.27)) hide)
     )
@@
       (effects (font (size 1.27 1.27)) (justify right))
     )
-    (property "Footprint" "Connector_JST:JST_XA_B04B-XASK-1-A_1x04_P2.50mm_Vertical" (at 205.74 106.68 0)
+    (property "Footprint" "Connector_JST:JST_XH_B4B-XH-A_1x04_P2.50mm_Vertical" (at 205.74 106.68 0)
       (effects (font (size 1.27 1.27)) hide)
     )
@@
       (effects (font (size 1.27 1.27)))
     )
-    (property "Footprint" "Connector_JST:JST_XA_B05B-XASK-1-A_1x05_P2.50mm_Vertical" (at 41.91 123.19 0)
+    (property "Footprint" "Connector_JST:JST_XH_B5B-XH-A_1x05_P2.50mm_Vertical" (at 41.91 123.19 0)
       (effects (font (size 1.27 1.27)) hide)
     )
@@
       (effects (font (size 1.27 1.27)))
     )
-    (property "Footprint" "Connector_JST:JST_XA_B03B-XASK-1-A_1x03_P2.50mm_Vertical" (at 153.67 134.62 0)
+    (property "Footprint" "Connector_JST:JST_XH_B3B-XH-A_1x03_P2.50mm_Vertical" (at 153.67 134.62 0)
       (effects (font (size 1.27 1.27)) hide)
     )
@@
       (effects (font (size 1.27 1.27)) (justify right))
     )
-    (property "Footprint" "Connector_JST:JST_XA_B03B-XASK-1-A_1x03_P2.50mm_Vertical" (at 184.15 109.22 0)
-      (effects (font (size 1.27 1.27)) hide)
-    )
+    (property "Footprint" "Connector_JST:JST_XH_B3B-XH-A_1x03_P2.50mm_Vertical" (at 184.15 109.22 0)
+      (effects (font (size 1.27 1.27)) hide)
+    )
