File: groundwork/Vim/new_pcb/arm_pcb/arm_pcb.kicad_pcb (KiCad board)
At the start: 2 copper layers, 81.3 x 61 mm, 18 parts, among them U1 NODEMCU32S

Commit message: pcb schematic udpate final v0.1
Parts:
- added REF**: MountingHole_4.3mm_M4, MountingHole:MountingHole_4.3mm_M4, F.Cu at (124.5, 121.9)
- added REF**: MountingHole_4.3mm_M4, MountingHole:MountingHole_4.3mm_M4, F.Cu at (53.3, 121.9)
- added REF**: MountingHole_4.3mm_M4, MountingHole:MountingHole_4.3mm_M4, F.Cu at (124.5, 71.1)
- added REF**: MountingHole_4.3mm_M4, MountingHole:MountingHole_4.3mm_M4, F.Cu at (53.3, 71.1)
- moved EncoderA3 34.2 mm to (116.8, 73.7), turned to 0 degrees
- moved Servo4 25.6 mm to (116.8, 109.2), turned to 0 degrees
- moved Servo3 25.6 mm to (104.2, 109.2), turned to 0 degrees
- moved Servo2 25.0 mm to (116.8, 99.1)
- moved Servo1 25.0 mm to (104.2, 99.1)
- moved EncoderA1 23.8 mm to (104.2, 73.7), turned to 0 degrees
- moved EncoderA4 21.4 mm to (116.9, 86.4), turned to 0 degrees
- moved EncoderA2 21.0 mm to (104.2, 86.4), turned to 0 degrees
- moved MotorDriver1 12.6 mm to (53.3, 81.3), turned to 0 degrees
- moved MotorDriver2 12.5 mm to (53.5, 91.4), turned to 0 degrees
- moved MotorDriver3 12.5 mm to (53.5, 101.6), turned to 0 degrees
- moved SPIBreakout1 8.03 mm to (61.0, 121.9), turned to 90 degrees
- moved MotorDriver4 7.62 mm to (53.5, 111.8)
- moved I2Cbreakout1 6.34 mm to (73.8, 71.1), turned to 0 degrees
- moved Stepper1 5.39 mm to (104.2, 119.4), turned to 0 degrees
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Connections:
- EncoderA1 pad 2: Net-(EncoderA1-Pin_2) -> a_in_1
- EncoderA2 pad 2: Net-(EncoderA2-Pin_2) -> a_in_2
- EncoderA3 pad 2: Net-(EncoderA3-Pin_2) -> a_in_3
- EncoderA4 pad 2: Net-(EncoderA4-Pin_2) -> a_in_4
- I2Cbreakout1 pad 3: Net-(I2Cbreakout1-Pin_3) -> servo3
- I2Cbreakout1 pad 4: Net-(I2Cbreakout1-Pin_4) -> servo4
- MotorDriver1 pad 2: Net-(MotorDriver1-Pin_2) -> m1_1
- MotorDriver1 pad 3: Net-(MotorDriver1-Pin_3) -> m1_2
- MotorDriver4 pad 2: Net-(MotorDriver4-Pin_2) -> SPI_MOSI
- MotorDriver4 pad 3: Net-(MotorDriver4-Pin_3) -> SPI_MISO
- MotorDriver4 pad 4: Net-(MotorDriver4-Pin_4) -> SPI_SCK
- MotorDriver4 pad 5: SPI_SCK -> m4_4
- Servo3 pad 2: Net-(Servo3-Pin_2) -> servo3
- Servo4 pad 2: Net-(Servo4-Pin_2) -> servo4
- Stepper1 pad 1: Net-(Stepper1-Pin_1) -> SPI_SCK
- U1 pad GPIO0: Net-(EncoderA3-Pin_2) -> m1_1
- U1 pad GPIO10: Net-(MotorDriver3-Pin_4) -> unconnected-(U1-PadGPIO10)
- U1 pad GPIO11: Net-(MotorDriver3-Pin_5) -> unconnected-(U1-PadGPIO11)
- U1 pad GPIO15: Net-(EncoderA4-Pin_2) -> Net-(MotorDriver3-Pin_4)
- U1 pad GPIO2: unconnected-(U1-PadGPIO2) -> m4_4
- U1 pad GPIO21: Net-(I2Cbreakout1-Pin_3) -> servo3
- U1 pad GPIO22: Net-(I2Cbreakout1-Pin_4) -> servo4
- U1 pad GPIO27: Net-(EncoderA1-Pin_2) -> Net-(MotorDriver3-Pin_3)
- U1 pad GPIO34: Net-(MotorDriver1-Pin_2) -> a_in_1
- U1 pad GPIO35: Net-(MotorDriver1-Pin_3) -> a_in_2
- U1 pad GPIO36: Net-(MotorDriver4-Pin_2) -> a_in_3
- U1 pad GPIO39: Net-(MotorDriver4-Pin_3) -> a_in_4
- U1 pad GPIO4: Net-(EncoderA2-Pin_2) -> m1_2
- U1 pad GPIO5: Net-(Stepper1-Pin_1) -> Net-(MotorDriver3-Pin_5)
- U1 pad GPIO6: Net-(MotorDriver4-Pin_4) -> unconnected-(U1-PadGPIO6)
- U1 pad GPIO7: Net-(Servo4-Pin_2) -> unconnected-(U1-PadGPIO7)
- U1 pad GPIO8: Net-(Servo3-Pin_2) -> unconnected-(U1-PadGPIO8)
- U1 pad GPIO9: Net-(MotorDriver3-Pin_3) -> unconnected-(U1-PadGPIO9)
Routing:
- net GND: track 279.0 -> 0.00 mm, vias 1 -> 0
- net m1_1: track 0.00 -> 68.3 mm
- net servo4: track 0.00 -> 66.7 mm
- net Net-(Servo4-Pin_2): track 59.4 -> 0.00 mm
- net m1_2: track 0.00 -> 59.3 mm
- net SPI_RST: track 0.00 -> 54.3 mm
- net servo3: track 0.00 -> 52.4 mm
- net a_in_3: track 0.00 -> 49.1 mm
- net Net-(Servo3-Pin_2): track 47.9 -> 0.00 mm
- net a_in_4: track 0.00 -> 46.1 mm
- net a_in_1: track 0.00 -> 45.4 mm
- net Net-(MotorDriver4-Pin_4): track 44.5 -> 0.00 mm
- net Net-(MotorDriver4-Pin_2): track 40.8 -> 0.00 mm
- net Net-(EncoderA1-Pin_2): track 39.1 -> 0.00 mm
- net m4_4: track 0.00 -> 36.4 mm
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Other:
- board text added: "Project Kratos"

Commit message: final pcb v0.2
Parts:
- removed REF** (x4): MountingHole_4.3mm_M4, MountingHole:MountingHole_4.3mm_M4
- added 5V_3V_jumper: JST_XH_B3B-XH-A_1x03_P2.50mm_Vertical, Connector_JST:JST_XH_B3B-XH-A_1x03_P2.50mm_Vertical, F.Cu at (229.9, 108.0)
- added G***: LOGO, LOGO, F.Cu at (238.1, 86.4)
- added mountinghole1: MountingHole_2.2mm_M2, MountingHole:MountingHole_2.2mm_M2, F.Cu at (157.5, 54.6)
- added mountinghole2: MountingHole_2.2mm_M2, MountingHole:MountingHole_2.2mm_M2, F.Cu at (157.5, 123.2)
- added mountinghole3: MountingHole_2.2mm_M2, MountingHole:MountingHole_2.2mm_M2, F.Cu at (240.0, 123.2)
- added mountinghole4: MountingHole_2.2mm_M2, MountingHole:MountingHole_2.2mm_M2, F.Cu at (240.0, 54.6)
- EncoderA1, EncoderA2, EncoderA3, EncoderA4, Servo1, Servo2, Servo3, Servo4, Stepper1, Stepper_GND1: footprint Connector_JST:JST_XA_B03B-XASK-1-A_1x03_P2.50mm_Vertical -> Connector_JST:JST_XH_B3B-XH-A_1x03_P2.50mm_Vertical
- I2Cbreakout1, UART0breakout1: footprint Connector_JST:JST_XA_B04B-XASK-1-A_1x04_P2.50mm_Vertical -> Connector_JST:JST_XH_B4B-XH-A_1x04_P2.50mm_Vertical
- MotorDriver1, MotorDriver2, MotorDriver3, MotorDriver4: footprint Connector_JST:JST_XA_B05B-XASK-1-A_1x05_P2.50mm_Vertical -> Connector_JST:JST_XH_B5B-XH-A_1x05_P2.50mm_Vertical
- moved MotorDriver4 186.1 mm to (231.0, 55.9), turned to 180 degrees
- moved MotorDriver3 164.9 mm to (211.9, 55.9), turned to 180 degrees
- moved SPIBreakout1 157.3 mm to (213.9, 85.1), turned to 180 degrees
- moved MotorDriver2 144.0 mm to (193.0, 55.9), turned to 180 degrees
- moved UART0breakout1 134.7 mm to (222.5, 89.3), turned to 90 degrees
- moved Stepper1 128.5 mm to (222.2, 68.6), turned to 180 degrees
- moved Stepper_GND1 128.0 mm to (234.4, 68.6), turned to 180 degrees
- moved MotorDriver1 123.3 mm to (174.0, 55.9), turned to 180 degrees
- moved EncoderA4 108.4 mm to (220.9, 116.8), turned to 180 degrees
- moved Servo4 104.4 mm to (221.0, 101.6), turned to 180 degrees
- moved Servo3 101.8 mm to (205.7, 101.6), turned to 180 degrees
- moved EncoderA3 98.8 mm to (205.7, 116.8), turned to 180 degrees
- moved U1 96.4 mm to (180.3, 78.7), turned to -90 degrees
- moved EncoderA2 91.5 mm to (190.5, 116.8), turned to 180 degrees
- moved I2Cbreakout1 91.4 mm to (157.5, 107.9), turned to 90 degrees
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Routing:
- net SPI_MOSI: track 112.4 -> 0.00 mm, vias 1 -> 0
- net SPI_MISO: track 100.8 -> 0.00 mm
- net SPI_SCK: track 84.6 -> 0.00 mm
- net m1_1: track 68.3 -> 0.00 mm
- net servo4: track 66.7 -> 0.00 mm
- net m1_2: track 59.3 -> 0.00 mm
- net SPI_RST: track 54.3 -> 0.00 mm
- net servo3: track 52.4 -> 0.00 mm
- net Net-(MotorDriver3-Pin_4): track 49.7 -> 0.00 mm
- net a_in_3: track 49.1 -> 0.00 mm
- net a_in_4: track 46.1 -> 0.00 mm
- net a_in_1: track 45.4 -> 0.00 mm
- net m4_4: track 36.4 -> 0.00 mm
- net Net-(MotorDriver3-Pin_5): track 36.2 -> 0.00 mm
- net a_in_2: track 34.4 -> 0.00 mm
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Other:
- board size 81.3 x 61 mm -> 91.4 x 76.2 mm
- board text added: "18 19 23"
- board text added: "3V3 GPIO34 GND"
- board text added: "3V3 GPIO35 GND"
- board text added: "3V3 GPIO36 GND"
- board text added: "3V3 GPIO39 GND"
- board text added: "GND 5V (Servo) 3V3"
- board text added: "GND MA1/0 MA2/4 MB1/32 MB2/33"
- board text added: "GND MA1/13 MA2/27 MB1/15 MB2/5"
- board text added: "GND MA1/23 MA2/19 MB1/18 MB2/2"
- board text added: "GND MA1/25 MA2/26 MB1/14 MB2/12"
- board text added: "GND MOSI VCC"
- board text added: "POWER GPIO16 GND"
- board text added: "POWER GPIO17 GND"
- board text added: "POWER GPIO21 GND"
- board text added: "POWER GPIO22 GND"
- board text added: "RST SCK MISO"
- board text added: "SCL/22 SDA/21 3V3 GND"
- board text added: "TX0/GPIO1 RX0/GPIO3 3V3 GND"
- board text removed: "Project Kratos"

Commit message: pcb almost done v0
Routing:
- net Net-(UART0breakout1-Pin_3): track 0.00 -> 137.4 mm, vias 0 -> 1
- net servo4: track 0.00 -> 136.2 mm, vias 0 -> 1
- net Net-(UART0breakout1-Pin_4): track 0.00 -> 126.1 mm, vias 0 -> 1
- net servo3: track 0.00 -> 109.9 mm
- net a_in_1: track 0.00 -> 90.2 mm, vias 0 -> 1
- net m4_4: track 0.00 -> 87.6 mm, vias 0 -> 1
- net Net-(MotorDriver3-Pin_4): track 0.00 -> 83.4 mm, vias 0 -> 1
- net SPI_MISO: track 0.00 -> 81.7 mm, vias 0 -> 3
- net SPI_SCK: track 0.00 -> 78.8 mm, vias 0 -> 1
- net SPI_MOSI: track 0.00 -> 76.2 mm
- net Net-(Servo2-Pin_2): track 0.00 -> 63.1 mm, vias 0 -> 1
- net Net-(MotorDriver3-Pin_5): track 0.00 -> 61.0 mm, vias 0 -> 2
- net Net-(MotorDriver3-Pin_2): track 0.00 -> 57.1 mm
- net Net-(MotorDriver3-Pin_3): track 0.00 -> 49.8 mm, vias 0 -> 1
- net Net-(Servo1-Pin_2): track 0.00 -> 41.1 mm
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- added copper zone on F.Cu, net VCCQ

Commit message: update v0.2
Parts:
- moved EncoderA1 16.6 mm to (177.0, 100.3)
- moved EncoderA2 16.6 mm to (192.3, 100.3)
- moved EncoderA3 16.6 mm to (207.5, 100.3)
- moved EncoderA4 16.6 mm to (222.7, 100.3)
- moved Servo1 14.3 mm to (177.0, 115.8)
- moved Servo2 14.3 mm to (192.2, 115.8)
- moved Servo3 14.3 mm to (207.4, 115.8)
- moved Servo4 14.3 mm to (222.7, 115.8)
- moved 5V_3V_jumper 6.14 mm to (234.7, 104.2), turned to -90 degrees
- renumbered G*** to KratosLogo
Routing:
- net Net-(UART0breakout1-Pin_3): track 137.4 -> 0.00 mm, vias 1 -> 0
- net servo4: track 136.2 -> 0.00 mm, vias 1 -> 0
- net Net-(UART0breakout1-Pin_4): track 126.1 -> 0.00 mm, vias 1 -> 0
- net servo3: track 109.9 -> 0.00 mm
- net a_in_1: track 90.2 -> 0.00 mm, vias 1 -> 0
- net m4_4: track 87.6 -> 0.00 mm, vias 1 -> 0
- net Net-(MotorDriver3-Pin_4): track 83.4 -> 0.00 mm, vias 1 -> 0
- net SPI_MISO: track 81.7 -> 0.00 mm, vias 3 -> 0
- net SPI_SCK: track 78.8 -> 0.00 mm, vias 1 -> 0
- net SPI_MOSI: track 76.2 -> 0.00 mm
- net Net-(Servo2-Pin_2): track 63.1 -> 0.00 mm, vias 1 -> 0
- net Net-(MotorDriver3-Pin_5): track 61.0 -> 0.00 mm, vias 2 -> 0
- net Net-(MotorDriver3-Pin_2): track 57.1 -> 0.00 mm
- net Net-(MotorDriver3-Pin_3): track 49.8 -> 0.00 mm, vias 1 -> 0
- net Net-(Servo1-Pin_2): track 41.1 -> 0.00 mm
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- removed copper zone on F.Cu, net VCCQ

Commit message: pcb done-ishhh
Routing:
- net VCCQ: track 117.8 -> 219.4 mm
- net servo4: track 0.00 -> 90.0 mm
- net servo3: track 0.00 -> 70.1 mm
- net m4_4: track 0.00 -> 69.8 mm
- net SPI_MISO: track 0.00 -> 69.8 mm
- net SPI_SCK: track 0.00 -> 67.5 mm
- net Net-(MotorDriver3-Pin_4): track 0.00 -> 62.7 mm
- net Net-(MotorDriver3-Pin_2): track 0.00 -> 59.6 mm
- net SPI_MOSI: track 0.00 -> 52.2 mm
- net a_in_4: track 0.00 -> 49.5 mm
- net Net-(MotorDriver3-Pin_5): track 0.00 -> 45.8 mm
- net a_in_1: track 0.00 -> 44.7 mm, vias 0 -> 1
- net m1_1: track 0.00 -> 41.4 mm
- net Net-(MotorDriver3-Pin_3): track 0.00 -> 40.1 mm
- net Net-(Servo2-Pin_2): track 0.00 -> 37.4 mm
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